Commit message: Исправил urdf

File: urdf/rars01.urdf (robot description, URDF)
Before this commit: robot rars01, 9 links, 8 joints
Links:
- link End_link: mass 0.35750000 -> 0.45
Joints:
- joint joint2: limit lower=0 upper=3.14 effort=27 velocity=10 -> lower=0 upper=3.6 effort=27 velocity=10
- joint joint4: limit lower=-1.4 upper=1.4 effort=7 velocity=10 -> lower=-2.0 upper=1.4 effort=7 velocity=10
