Commit message: final urdf version

File: source/solidworks_export/urdf/RARS01_1.urdf (robot description, URDF)
Before this commit: robot RARS01_1, 9 links, 8 joints
Links:
- removed link link_6_m6
- added link gripper_left, mass 0.08529926; collision mesh filename=package://rars01_description/meshes/gripper_left.STL; visual mesh filename=package://rars01_description/meshes/gripper_left.STL
- added link gripper_right, mass 0.08529926; collision mesh filename=package://rars01_description/meshes/gripper_right.STL; visual mesh filename=package://rars01_description/meshes/gripper_right.STL
- link End_link: mass 0.35750000 -> 0.60527119; geometry collision mesh filename=package://rars01_description/meshes/End_link.STL; visual mesh filename=package://rars01_description/meshes/End_link.STL
- link base_link: geometry collision mesh filename=package://rars01_description/meshes/base_link.STL; visual mesh filename=package://rars01_description/meshes/base_link.STL
- link link1_m0: geometry collision mesh filename=package://rars01_description/meshes/link1_m0.STL; visual mesh filename=package://rars01_description/meshes/link1_m0.STL
- link link2_m1: geometry collision mesh filename=package://rars01_description/meshes/link2_m1.STL; visual mesh filename=package://rars01_description/meshes/link2_m1.STL
- link link2_m2: geometry collision mesh filename=package://rars01_description/meshes/link2_m2.STL; visual mesh filename=package://rars01_description/meshes/link2_m2.STL
- link link_3_m3: geometry collision mesh filename=package://rars01_description/meshes/link_3_m3.STL; visual mesh filename=package://rars01_description/meshes/link_3_m3.STL
- link link_4_m4: geometry collision mesh filename=package://rars01_description/meshes/link_4_m4.STL; visual mesh filename=package://rars01_description/meshes/link_4_m4.STL
- link link_5_m5: geometry collision mesh filename=package://rars01_description/meshes/link_5_m5.STL; visual mesh filename=package://rars01_description/meshes/link_5_m5.STL
Joints:
- removed joint joint0
- added joint gripper_left_joint: type prismatic, parent End_link, child gripper_left, origin xyz=-0.0375 0 0 rpy=0 0 0, axis 0 1 0, limit lower=0 upper=0.05 effort=3 velocity=10
- added joint gripper_right_joint: type prismatic, parent End_link, child gripper_right, origin xyz=-0.0375000000000192 0 0 rpy=0 0 0, axis 0 -1 0, limit lower=0 upper=0.05 effort=3 velocity=10, mimic joint=gripper_left_joint multiplier=1 offset=0
- joint joint1: axis 0 1 0 -> 0 0 1; child link2_m1 -> link1_m0; limit lower=0 upper=3.14 effort=27 velocity=10 -> lower=-2.8 upper=2.8 effort=27 velocity=10; origin xyz=0.02 -0.029675 0.075 rpy=0 0 0 -> xyz=0 0 0.0643 rpy=0 0 0; parent link1_m0 -> base_link
- joint joint2: axis 0 -1 0 -> 0 1 0; child link2_m2 -> link2_m1; limit lower=0 upper=3.14 effort=27 velocity=10 -> lower=0 upper=3.6 effort=27 velocity=10; origin xyz=-0.250000000000001 0 0 rpy=0 0 0 -> xyz=0.02 -0.029675 0.075 rpy=0 0 0; parent link2_m1 -> link1_m0
- joint joint3: child link_3_m3 -> link2_m2; limit lower=-1.4 upper=1.4 effort=7 velocity=10 -> lower=0 upper=3.14 effort=27 velocity=10; origin xyz=0.232950000000001 0.00377499999999996 0.0570710741093906 rpy=0 0 0 -> xyz=-0.250000000000001 0 0 rpy=0 0 0; parent link2_m2 -> link2_m1
- joint joint4: axis 0 0 -1 -> 0 -1 0; child link_4_m4 -> link_3_m3; limit lower=-1.57 upper=1.57 effort=7 velocity=10 -> lower=-2.0 upper=1.4 effort=7 velocity=10; origin xyz=0.0798112070633211 0.0260499999999993 0.0499999999999984 rpy=0 0 0 -> xyz=0.232950000000001 0.00377499999999996 0.0570710741093906 rpy=0 0 0; parent link_3_m3 -> link2_m2
- joint joint5: axis 1 0 0 -> 0 0 -1; child link_5_m5 -> link_4_m4; limit lower=-2 upper=2 effort=7 velocity=0 -> lower=-1.57 upper=1.57 effort=7 velocity=10; origin xyz=0.0235 0 -0.049 rpy=0 0 0 -> xyz=0.0798112070633211 0.0260499999999993 0.0499999999999984 rpy=0 0 0; parent link_4_m4 -> link_3_m3
- joint joint6: axis 0 -1 0 -> 1 0 0; child link_6_m6 -> link_5_m5; limit lower=0 upper=1.4 effort=0 velocity=0 -> lower=-2 upper=2 effort=7 velocity=10; origin xyz=-0.13 -0.0255 0 rpy=0 0 0 -> xyz=0.0235 0 -0.049 rpy=0 0 0; parent End_link -> link_4_m4
- joint joint_end: axis 0 0 0 -> (none); limit lower=1 upper=0 effort=7 velocity=0 -> (none); origin xyz=0.18 0 0 rpy=0 0 0 -> xyz=0.195000000000023 0 0 rpy=0 0 0

File: urdf/rars01.urdf (robot description, URDF)
Before this commit: robot rars01, 9 links, 8 joints
Links:
- removed link link_6_m6
- added link gripper_left, mass 0.08529926; collision mesh filename=package://rars01_description/meshes/gripper_left.STL; visual mesh filename=package://rars01_description/meshes/gripper_left.STL
- added link gripper_right, mass 0.08529926; collision mesh filename=package://rars01_description/meshes/gripper_right.STL; visual mesh filename=package://rars01_description/meshes/gripper_right.STL
- link End_link: mass 0.45 -> 0.60527119
Joints:
- removed joint gripper
- added joint gripper_left_joint: type prismatic, parent End_link, child gripper_left, origin xyz=-0.0375 0 0 rpy=0 0 0, axis 0 1 0, limit lower=0 upper=0.05 effort=3 velocity=10
- added joint gripper_right_joint: type prismatic, parent End_link, child gripper_right, origin xyz=-0.0375000000000192 0 0 rpy=0 0 0, axis 0 -1 0, limit lower=0 upper=0.05 effort=3 velocity=10, mimic joint=gripper_left_joint multiplier=1 offset=0
- joint joint_end: origin xyz=0.18 0 0 rpy=0 0 0 -> xyz=0.195000000000023 0 0 rpy=0 0 0
